File: elec/main.sch (EAGLE design)
At the start: 9 parts, among them IC1 NE556D, IC2 4066D

Commit message: Elec
Parts:
- removed C3, C4: (no value), rcl:C-EUC0805
- added C5: (no value), rcl:CPOL-EUE2,5-6E
- added D1: 1N4004, diode:1N4004
- added D2: 1N4148, diode:1N4148DO35-7
- added LD1: (no value), led:DUOLED-RG-C
- added R10: 22k, rcl:R-EU_R0805
- added R11, R12, R6, R7, R9: (no value), rcl:R-EU_R0805
- added R4: 22k, pot:TRIM_EU-RJ6
- added R5: 10k, rcl:R-EU_R0805
- added R8: 1k, rcl:R-EU_R0805
- added S1, S2: DT6, switch-misc:DT6
- added S3: (no value), switch:320-916
- added SV1: (no value), con-lsta:FE08-1
- added SV2, SV3: (no value), con-lstb:MA04-1
- added T1: 2N2222, transistor:2N2222
- added X1: (no value), con-wago-500:W237-102
- C2: value (none) -> 100nf
- R1: value (none) -> 2.2k
- R2, R3: value (none) -> 10k
Connections:
- new net FORCE: IC1B.THR, IC1B.TR, IC2A.A, R3.1, R5.2, SV1.3
- new net N$10: D1.A, T1.C, X1-1.KL
- new net N$11: R11.2, S1.P, S1.P@1
- new net N$12: R7.1, T1.B
- new net N$13: D2.A, IC1A.Q
- new net N$14: LD1.C, R9.1
- new net N$15: IC2C.A, LD1.AG
- new net N$17: IC2B.B, IC2C.C, R10.1
- new net N$19: R12.1, S2.S, S2.S@1
- new net N$3: R1.1, R4.S
- new net N$6: SV2.3
- new net N$7: SV2.4
- new net N$8: C5.+, IC2A.B, R6.1
- new net R_FORCE: S1.S, S1.S@1, S2.P, S2.P@1, SV3.1
- new net R_TIP_IN: S3.O, SV3.2
- new net STATE: IC1B.Q, IC2B.C, LD1.AR, R6.2, R7.2, SV1.4
- new net SWITCH: D2.C, IC2A.C, R8.1, SV1.5
- new net TIP: IC1A.TR, R2.1, SV2.1
- new net TIP_IN: SV1.6, SV2.2
- net GND: now also C5.-, IC2B.A, R11.1, R2.2, R5.1, R8.2, R9.2, SV1.1, SV1.7, SV3.4, T1.E
- net VCC: now also D1.C, IC2C.B, R10.2, R12.2, R3.2, R4.E, S3.P, SV1.2, SV1.8, SV3.3, X1-2.KL
Other:
- note added: "ManualPickAndPlace"
- note added: "Remote"
- note added: "hugo, 07/2014"
- moved on the sheet: IC1B, IC2A, IC2B, IC2C, R1, R2, R3
